File: PCB/Mirza.kicad_pcb (KiCad board)
At the start: 2 copper layers, 17 parts, among them Q1 BC857BS, Q10 BC847BS, Q11 BCX56, Q12 BCX53, Q13 BCX56, Q14 BCX53, Q15 BCX56, Q16 BCX53, Q2 BC847BS, Q3 BCX56, Q4 BCX53, Q5 BCX56, Q6 BCX53, Q7 BCX56, Q8 BCX53, Q9 BC857BS

Commit message: Completed layout
Parts:
- removed L1: 78602/3JC, Ariamelon-Device:L_Murata_786J
- added A1: Ariamelon Logo, Ariamelon-Logo:Ariamelon_Logo_Small_CU, F.Cu at (131.8, 51.1)
- added C1: 100p, Ariamelon-Device:C_0805_2012Metric, F.Cu at (79.2, 65.8)
- added C10: 1u, Ariamelon-Device:C_0805_2012Metric, F.Cu at (94.6, 71.4)
- added C11: 1u, Ariamelon-Device:C_0805_2012Metric, F.Cu at (91.1, 66.7)
- added C12: 100u, Capacitor_THT:CP_Radial_D6.3mm_P2.50mm, F.Cu at (134.4, 60.7)
- added C13: 100u, Capacitor_THT:CP_Radial_D6.3mm_P2.50mm, F.Cu at (134.4, 70.2)
- added C14: 100u, Capacitor_THT:CP_Radial_D6.3mm_P2.50mm, F.Cu at (141.4, 60.7)
- added C15: 100u, Capacitor_THT:CP_Radial_D6.3mm_P2.50mm, F.Cu at (141.4, 70.2)
- added C16: 100n, Ariamelon-Device:C_0805_2012Metric, F.Cu at (96.3, 61.9)
- added C17: 100n, Ariamelon-Device:C_0805_2012Metric, F.Cu at (98.4, 71.4)
- added C18: 68u, Capacitor_THT:CP_Radial_D5.0mm_P2.00mm, F.Cu at (106.1, 52.0)
- added C19: 68u, Capacitor_THT:CP_Radial_D5.0mm_P2.00mm, F.Cu at (94.5, 52.0)
- added C2: 47p, Ariamelon-Device:C_0805_2012Metric, F.Cu at (101.7, 59.8)
- added C20: 68u, Capacitor_THT:CP_Radial_D5.0mm_P2.00mm, F.Cu at (92.5, 81.4)
- added C21: 68u, Capacitor_THT:CP_Radial_D5.0mm_P2.00mm, F.Cu at (104.1, 81.4)
- added C3: 47p, Ariamelon-Device:C_0805_2012Metric, F.Cu at (101.7, 73.6)
- added C4: 100p, Ariamelon-Device:C_0805_2012Metric, F.Cu at (105.8, 59.8)
- added C5: 100p, Ariamelon-Device:C_0805_2012Metric, F.Cu at (105.8, 73.6)
- added C6: 47p, Ariamelon-Device:C_0805_2012Metric, F.Cu at (106.8, 62.6)
- added C7: 100p, Ariamelon-Device:C_0805_2012Metric, F.Cu at (118.9, 61.0)
- added C8: 100p, Ariamelon-Device:C_0805_2012Metric, F.Cu at (118.9, 72.4)
- added C9: 100p, Ariamelon-Device:C_0805_2012Metric, F.Cu at (138.3, 66.7)
- added D1: 1N4148W, Ariamelon-Device:D_SOD-123, F.Cu at (129.5, 61.1)
- added D2: 1N4148W, Ariamelon-Device:D_SOD-123, F.Cu at (129.5, 72.3)
- added H1: Star Ground, TestPoint:TestPoint_THTPad_D2.0mm_Drill1.0mm, F.Cu at (106.8, 65.7)
- added H2: M3, MountingHole:MountingHole_3.2mm_M3_Pad, F.Cu at (77.6, 52.4)
- added H3: M3, MountingHole:MountingHole_3.2mm_M3_Pad, F.Cu at (77.6, 81.0)
- added H4: M3, MountingHole:MountingHole_3.2mm_M3_Pad, F.Cu at (146.5, 81.0)
- added H5: M3, MountingHole:MountingHole_3.2mm_M3_Pad, F.Cu at (146.5, 52.4)
- added J1: In, Connector_PinHeader_2.54mm:PinHeader_1x02_P2.54mm_Vertical, F.Cu at (75.8, 68.0)
- added J2: Out, Connector_PinHeader_2.54mm:PinHeader_1x02_P2.54mm_Vertical, F.Cu at (129.5, 68.0)
- added J3: Power, Ariamelon-Header:PinHeader_1x04_P2.54mm_Vertical_MiddleGND, F.Cu at (148.3, 66.7)
- added Q17: 2SC3324, Ariamelon-Package:SOT-23-3, F.Cu at (109.9, 71.4)
- added Q18: 2SC3324, Ariamelon-Package:SOT-23-3, F.Cu at (107.5, 76.6)
- added Q19: PMP4201Y, Ariamelon-Package:SOT-363_SC-70-6, F.Cu at (110.0, 51.7)
- added Q20: PMP5201Y, Ariamelon-Package:SOT-363_SC-70-6, F.Cu at (119.0, 58.2)
- added Q21: PMP4201Y, Ariamelon-Package:SOT-363_SC-70-6, F.Cu at (118.9, 75.2)
- added Q22: 2SA1312, Ariamelon-Package:SOT-23-3, F.Cu at (114.3, 64.3)
- added Q23: 2SC3324, Ariamelon-Package:SOT-23-3, F.Cu at (114.3, 69.1)
- added Q24: 2SC3324, Ariamelon-Package:SOT-23-3, F.Cu at (118.9, 64.3)
- added Q25: 2SA1312, Ariamelon-Package:SOT-23-3, F.Cu at (118.9, 69.1)
- added Q26: D45H11, Ariamelon-Package:TO-220-3_Horizontal_TabUp, B.Cu at (123.2, 54.2)
- added Q27: D44H11, Ariamelon-Package:TO-220-3_Horizontal_TabUp, B.Cu at (123.2, 79.2)
- added Q28: PMP5201Y, Ariamelon-Package:SOT-363_SC-70-6, F.Cu at (110.0, 81.6)
- added R1: 2k2, Resistor_SMD:R_MiniMELF_MMA-0204, F.Cu at (77.3, 62.3)
- added R10: 560, Resistor_SMD:R_MiniMELF_MMA-0204, F.Cu at (93.5, 75.1)
- added R11: 560, Resistor_SMD:R_MiniMELF_MMA-0204, F.Cu at (96.1, 58.3)
- added R12: 68, Resistor_SMD:R_MiniMELF_MMA-0204, F.Cu at (88.1, 64.0)
- added R13: 68, Resistor_SMD:R_MiniMELF_MMA-0204, F.Cu at (88.1, 69.4)
- added R14: 560, Resistor_SMD:R_MiniMELF_MMA-0204, F.Cu at (98.7, 75.1)
- added R15: 2k2, Resistor_SMD:R_MiniMELF_MMA-0204, F.Cu at (102.6, 61.9)
- added R16: 2k2, Resistor_SMD:R_MiniMELF_MMA-0204, F.Cu at (102.6, 71.5)
- added R17: 220, Resistor_SMD:R_MiniMELF_MMA-0204, F.Cu at (98.7, 58.3)
- added R18: 220, Resistor_SMD:R_MiniMELF_MMA-0204, F.Cu at (110.5, 56.8)
- added R19: 100k, Resistor_SMD:R_MiniMELF_MMA-0204, F.Cu at (110.8, 66.7)
- added R2: 68, Resistor_SMD:R_MiniMELF_MMA-0204, F.Cu at (80.6, 68.0)
- added R20: 220, Resistor_SMD:R_MiniMELF_MMA-0204, F.Cu at (110.5, 76.6)
- added R21: 220, Resistor_SMD:R_MiniMELF_MMA-0204, F.Cu at (96.1, 75.1)
- added R22: 2k2, Resistor_SMD:R_MiniMELF_MMA-0204, F.Cu at (112.9, 51.7)
- added R23: 1M, Resistor_SMD:R_MiniMELF_MMA-0204, F.Cu at (106.8, 69.8)
- added R24: 100k, Resistor_SMD:R_MiniMELF_MMA-0204, F.Cu at (121.9, 66.7)
- added R25: 220, Resistor_SMD:R_MiniMELF_MMA-0204, F.Cu at (114.3, 57.9)
- added R26: 68, Resistor_SMD:R_MiniMELF_MMA-0204, F.Cu at (114.3, 60.7)
- added R27: 68, Resistor_SMD:R_MiniMELF_MMA-0204, F.Cu at (114.3, 72.7)
- added R28: 220, Resistor_SMD:R_MiniMELF_MMA-0204, F.Cu at (114.3, 75.5)
- added R29: 220, Resistor_SMD:R_MiniMELF_MMA-0204, F.Cu at (120.7, 52.9)
- added R3: 100k, Resistor_SMD:R_MiniMELF_MMA-0204, F.Cu at (80.6, 70.5)
- added R30: 220, Resistor_SMD:R_MiniMELF_MMA-0204, F.Cu at (120.7, 80.5)
- added R31: 0R33, Resistor_SMD:R_MELF_MMB-0207, F.Cu at (126.0, 62.9)
- added R32: 0R33, Resistor_SMD:R_MELF_MMB-0207, F.Cu at (126.0, 70.5)
- added R33: 68, Resistor_SMD:R_MiniMELF_MMA-0204, F.Cu at (134.1, 66.7)
- added R34: 1M, Resistor_SMD:R_MiniMELF_MMA-0204, F.Cu at (91.1, 70.8)
- added R35: 1M, Resistor_SMD:R_MiniMELF_MMA-0204, F.Cu at (102.6, 69.1)
- added R36: 560, Resistor_SMD:R_MiniMELF_MMA-0204, F.Cu at (102.6, 64.3)
- added R37: 150, Resistor_SMD:R_MiniMELF_MMA-0204, F.Cu at (102.6, 66.7)
- added R38: 100k, Resistor_SMD:R_MiniMELF_MMA-0204, F.Cu at (91.1, 62.6)
- added R39: 2k2, Resistor_SMD:R_MiniMELF_MMA-0204, F.Cu at (112.9, 81.6)
- added R4: 100k, Resistor_SMD:R_MiniMELF_MMA-0204, F.Cu at (82.0, 64.2)
- added R5: 560, Resistor_SMD:R_MiniMELF_MMA-0204, F.Cu at (93.5, 58.3)
- added R6: 68, Resistor_SMD:R_MiniMELF_MMA-0204, F.Cu at (85.0, 55.2)
- added R7: 10, Resistor_SMD:R_MiniMELF_MMA-0204, F.Cu at (82.0, 59.0)
- added R8: 10, Resistor_SMD:R_MiniMELF_MMA-0204, F.Cu at (82.0, 74.3)
- added R9: 68, Resistor_SMD:R_MiniMELF_MMA-0204, F.Cu at (85.0, 78.1)
- added RV1: 1k, Potentiometer_THT:Potentiometer_Bourns_3266W_Vertical, F.Cu at (115.5, 50.4)
- added RV2: 1k, Potentiometer_THT:Potentiometer_Bourns_3266W_Vertical, F.Cu at (118.0, 83.0)
- added U1: OPA604, Ariamelon-Package:SOIC-8_3.9x4.9mm_P1.27mm, F.Cu at (96.0, 66.7)
- Q1, Q9: value BC857BS -> PMP5201Y; footprint Package_TO_SOT_SMD:SOT-363_SC-70-6 -> Ariamelon-Package:SOT-363_SC-70-6
- Q10: value BC847BS -> PMP5201Y; footprint Package_TO_SOT_SMD:SOT-363_SC-70-6 -> Ariamelon-Package:SOT-363_SC-70-6
- Q11: value BCX56 -> PMP4201Y; footprint Package_TO_SOT_SMD:SOT-89-3 -> Ariamelon-Package:SOT-363_SC-70-6
- Q12: value BCX53 -> PMP4201Y; footprint Package_TO_SOT_SMD:SOT-89-3 -> Package_TO_SOT_SMD:SOT-363_SC-70-6
- Q13, Q5: value BCX56 -> 2SC3324; footprint Package_TO_SOT_SMD:SOT-89-3 -> Ariamelon-Package:SOT-23-3
- Q14, Q16, Q8: value BCX53 -> 2SA1312; footprint Package_TO_SOT_SMD:SOT-89-3 -> Ariamelon-Package:SOT-23-3
- Q15, Q3, Q7: value BCX56 -> 2SA1312; footprint Package_TO_SOT_SMD:SOT-89-3 -> Ariamelon-Package:SOT-23-3
- Q2: value BC847BS -> PMP4201Y; footprint Package_TO_SOT_SMD:SOT-363_SC-70-6 -> Ariamelon-Package:SOT-363_SC-70-6
- Q4, Q6: value BCX53 -> 2SC3324; footprint Package_TO_SOT_SMD:SOT-89-3 -> Ariamelon-Package:SOT-23-3
- moved Q6 58.5 mm to (85.0, 59.6), turned to 90 degrees
- moved Q9 57.7 mm to (97.8, 53.6), turned to -90 degrees
- moved Q10 56.0 mm to (100.8, 53.6), turned to 90 degrees
- moved Q15 55.5 mm to (107.5, 56.8), turned to 90 degrees
- moved Q7 55.0 mm to (85.0, 73.7), turned to 90 degrees
- moved Q16 54.3 mm to (109.9, 62.0), turned to -90 degrees
- moved Q1 53.7 mm to (89.2, 54.8), turned to 90 degrees
- moved Q8 53.2 mm to (89.2, 75.1), turned to 180 degrees
- moved Q5 52.6 mm to (89.2, 58.2), turned to 180 degrees
- moved Q2 52.1 mm to (89.2, 78.5), turned to -90 degrees
- moved Q4 51.6 mm to (85.0, 69.0), turned to 90 degrees
- moved Q13 51.5 mm to (103.4, 57.1), turned to 180 degrees
- moved Q3 51.4 mm to (85.0, 64.4), turned to 90 degrees
- moved Q12 50.8 mm to (97.8, 79.8), turned to 90 degrees
- moved Q11 48.7 mm to (100.8, 79.7), turned to 90 degrees
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Connections:
- Q1 pad 3: Net-(D1-A) -> Net-(Q1B-C2)
- Q10 pad 1: VEE -> Net-(Q10A-E1)
- Q10 pad 3: Net-(D8-K) -> Net-(Q10B-C2)
- Q10 pad 4: Net-(Q10A-B1) -> Net-(Q10B-E2)
- Q10 pad 5: Net-(Q10A-C1) -> Net-(Q10A-B1)
- Q10 pad 6: Net-(Q10A-C1) -> Net-(Q10A-B1)
- Q11 pad 1: Net-(Q11-B) -> Net-(Q11A-E1)
- Q11 pad 2: VCC -> Net-(Q11A-B1)
- Q11 pad 3: Net-(Q11-E) -> Net-(Q11B-C2)
- Q12 pad 2: VEE -> Net-(Q11B-E2)
- Q12 pad 3: Net-(Q12-E) -> Net-(Q11A-E1)
- Q13 pad 1: Net-(Q13-B) -> Net-(Q10A-B1)
- Q13 pad 2: VCC -> Net-(Q10B-C2)
- Q14 pad 1: Net-(Q14-B) -> Net-(Q11A-B1)
- Q14 pad 2: VEE -> Net-(Q11B-C2)
- Q15 pad 1: Net-(Q15-B) -> Net-(Q13-E)
- Q15 pad 2: VCC -> Net-(Q15-C)
- Q15 pad 3: Net-(Q15-E) -> Net-(Q10B-C2)
- Q16 pad 2: VEE -> Net-(Q16-C)
- Q16 pad 3: Net-(Q16-E) -> Net-(Q15-C)
- Q2 pad 3: Net-(D4-K) -> Net-(Q2B-C2)
- Q3 pad 2: VCC -> Net-(Q3-C)
- Q4 pad 1: Net-(Q4-B) -> Net-(Q3-B)
- Q4 pad 2: VEE -> Net-(Q4-C)
- Q5 pad 1: Net-(Q5-B) -> Net-(Q1B-C2)
- Q5 pad 2: VCC -> Net-(Q10A-B1)
- Q6 pad 2: VEE -> Net-(Q5-E)
- Q6 pad 3: Net-(Q6-E) -> Net-(Q4-C)
- Q7 pad 2: VCC -> Net-(Q7-C)
- Q7 pad 3: Net-(Q7-E) -> Net-(Q3-C)
- Q8 pad 1: Net-(Q8-B) -> Net-(Q2B-C2)
- Q8 pad 2: VEE -> Net-(Q11A-B1)
- Q8 pad 3: Net-(Q8-E) -> Net-(Q7-C)
- Q9 pad 1: VCC -> Net-(Q9A-E1)
- Q9 pad 2: Net-(Q9A-B1) -> Net-(Q10B-E2)
- Q9 pad 3: Net-(D5-A) -> Net-(Q10A-E1)
- Q9 pad 4: Net-(Q9A-B1) -> Net-(Q9B-E2)
- Q9 pad 5: Net-(Q9A-C1) -> Net-(Q10B-E2)
- Q9 pad 6: Net-(Q9A-C1) -> Net-(Q10B-E2)
Routing:
- net Amp_Out: track 0.00 -> 40.0 mm, vias 0 -> 1
- net VCC: track 0.00 -> 32.0 mm, vias 0 -> 2
- net -18V: track 0.00 -> 30.1 mm, vias 0 -> 3
- net VEE: track 0.00 -> 30.0 mm, vias 0 -> 2
- net Amp_FB: track 0.00 -> 24.7 mm
- net Net-(Q2A-C1): track 0.00 -> 23.5 mm
- net Net-(Q16-C): track 0.00 -> 23.1 mm
- net Net-(Q10A-B1): track 0.00 -> 22.0 mm
- net +18V: track 0.00 -> 20.8 mm, vias 0 -> 2
- net Net-(Q11A-B1): track 0.00 -> 20.3 mm
- net Net-(Q23-C): track 0.00 -> 19.8 mm
- net Net-(Q24-C): track 0.00 -> 18.5 mm, vias 0 -> 1
- net Net-(Q1A-C1): track 0.00 -> 17.9 mm
- net Net-(Q25-E): track 0.00 -> 17.1 mm
- net Net-(Q22-C): track 0.00 -> 15.7 mm, vias 0 -> 2
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- added copper zone on F.Cu, net +18V
- added copper zone on F.Cu, net -18V
- added copper zone on F.Cu, net Amp_Out
- added copper zone on B.Cu, net GND
- added copper zone on F.Cu, net GND
- added copper zone on F.Cu, net Net-(C9-Pad2)
- added copper zone on F.Cu, net Net-(Q22-C)
- added copper zone on F.Cu, net Net-(Q23-C)
- added copper zone on F.Cu, net VCC
- added copper zone on F.Cu, net VEE
Other:
- board outline added: 75.9 x 35.6 mm
- board text added: "+18V"
- board text added: "-18V"
- board text added: "Bias"
- board text added: "G"
- board text added: "Mirza V1.0"
- board text added: "∿"
