File: PCB/Mirza.kicad_sch (KiCad schematic)
At the start: 8 parts, among them J1 Audio_In, J2 Audio_Out

Commit message: Completed layout
Parts:
- removed C25, C26: 150p, symbol Device:C_Small
- removed J1: Audio_In, symbol Ariamelon-Connector:Conn_Coaxial_x2_Dual_Separate_Small
- removed J2: Audio_Out, symbol Connector_Audio:AudioJack3
- removed L1: 78602/3JC, Ariamelon-Device:L_Murata_786J, symbol Ariamelon-Device:L_Coupled_Small_1{colon}1{colon}1
- removed R25, R26: 2k2, symbol Device:R_Small
- removed RV1: 10k, symbol Ariamelon-Device:R_Potentiometer_Dual_Separate_Small
- added A1: Ariamelon Logo, Ariamelon-Logo:Ariamelon_Logo_Small_CU, symbol Mechanical:Fiducial
- added C1, C2: 1u, Ariamelon-Device:C_0805_2012Metric, symbol Device:C_Small
- added C10, C6, C7: 47p, Ariamelon-Device:C_0805_2012Metric, symbol Device:C_Small
- added C101, C11, C12, C8 (x2), C9: 100p, Ariamelon-Device:C_0805_2012Metric, symbol Device:C_Small
- added C14 (x4): 68u, Capacitor_THT:CP_Radial_D5.0mm_P2.00mm, symbol Device:C_Polarized_Small
- added C14, C15, C17, C18: 100u, Capacitor_THT:CP_Radial_D6.3mm_P2.50mm, symbol Device:C_Polarized_Small
- added C3, C4: 100n, Ariamelon-Device:C_0805_2012Metric, symbol Device:C_Small
- added D1, D2: 1N4148W, Ariamelon-Device:D_SOD-123, symbol Device:D_Small
- added F1, F2: 500mA, Ariamelon-Device:Fuse_1206_3216Metric, symbol Device:Polyfuse_Small
- added H1: Star Ground, TestPoint:TestPoint_THTPad_D2.0mm_Drill1.0mm, symbol Ariamelon-Misc:MountingHole_Pad
- added H2, H3, H4, H5: M3, MountingHole:MountingHole_3.2mm_M3_Pad, symbol Mechanical:MountingHole
- added J1: In, Connector_PinHeader_2.54mm:PinHeader_1x02_P2.54mm_Vertical, symbol Connector_Generic:Conn_01x02
- added J2: Out, Connector_PinHeader_2.54mm:PinHeader_1x02_P2.54mm_Vertical, symbol Connector_Generic:Conn_01x02
- added J3: Power, Ariamelon-Header:PinHeader_1x04_P2.54mm_Vertical_MiddleGND, symbol Connector_Generic:Conn_01x04
- added Q1 (x5): PMP5201Y, Ariamelon-Package:SOT-363_SC-70-6, symbol Transistor_BJT:BC857BS
- added Q13, Q17, Q18, Q22, Q23, Q4, Q5, Q6: 2SC3324, Ariamelon-Package:SOT-23-3, symbol Device:Q_NPN_BCE
- added Q14, Q15, Q16, Q21, Q24, Q3, Q7, Q8: 2SA1312, Ariamelon-Package:SOT-23-3, symbol Device:Q_PNP_BCE
- added Q2 (x4): PMP4201Y, Ariamelon-Package:SOT-363_SC-70-6, symbol Transistor_BJT:BC847BS
- added Q2: PMP4201Y, Package_TO_SOT_SMD:SOT-363_SC-70-6, symbol Transistor_BJT:BC847BS
- added Q25: D45H11, Ariamelon-Package:TO-220-3_Horizontal_TabUp, symbol Device:Q_PNP_BCE
- added Q26: D44H11, Ariamelon-Package:TO-220-3_Horizontal_TabUp, symbol Device:Q_NPN_BCE
- added R1 (x2): 10, Resistor_SMD:R_MiniMELF_MMA-0204, symbol Device:R_Small
- added R1, R101 (x2), R6 (x4): 100k, Resistor_SMD:R_MiniMELF_MMA-0204, symbol Device:R_Small
- added R1 (x8): 68, Resistor_SMD:R_MiniMELF_MMA-0204, symbol Device:R_Small
- added R1, R5 (x3), R8: 560, Resistor_SMD:R_MiniMELF_MMA-0204, symbol Device:R_Small
- added R1 (x4), R5 (x4): 220, Resistor_SMD:R_MiniMELF_MMA-0204, symbol Device:R_Small
- added R1: 150, Resistor_SMD:R_MiniMELF_MMA-0204, symbol Device:R_Small
- added R1 (x2): 0R33, Resistor_SMD:R_MELF_MMB-0207, symbol Device:R_Small
- added R101, R6 (x2): 2k2, Resistor_SMD:R_MiniMELF_MMA-0204, symbol Device:R_Small
- added R6 (x3): 1M, Resistor_SMD:R_MiniMELF_MMA-0204, symbol Device:R_Small
- added RV2, RV3: 1k, Potentiometer_THT:Potentiometer_Bourns_3266W_Vertical, symbol Device:R_Potentiometer_Small
- added U1: OPA604, Ariamelon-Package:SOIC-8_3.9x4.9mm_P1.27mm, symbol Ariamelon-IC:Opamp_Single
Connections:
- net GND: now also C10.2, C101.1, C14.1, C14.1, C14.2, C14.2, C14.2, C15.2, C17.1, C18.1, C2.1, C3.2, C4.2, C8.1, H1.1, J1.1 (Pin_1), J2.1 (Pin_1), J3.2 (Pin_2), J3.3 (Pin_3), R1.2, R6.1, R6.1, R6.2
- new net: F1.1, J3.1 (Pin_1)
- new net: Q3.1 (B), Q4.1 (B), R1.2, R6.1
- new net: Q3.3 (E), R1.1
- new net: Q6.1 (B), R1.1, R1.2
- new net: C1.2, R1.1, U1.6
- new net: Q13.3 (E), Q15.1 (B), R5.1
- new net: Q16.1 (B), R5.2, R6.2
- new net: Q21.3 (E), R1.1
- new net: C11.1, Q1.3 (C2), Q23.1 (B), R1.2
- new net: C101.2, R1.1, R101.1
- new net: J1.2 (Pin_2), R101.2
- new net: Q1.2 (B1), Q1.4 (E2), R5.2 (x2)
- new net: Q1.5 (B2), Q1.6 (C1), R6.2 (x2)
- new net: C7.1, C9.1, R6.1
- new net: C10.1, C8.2, C9.2, Q16.2 (C), Q17.2 (C), Q21.1 (B), Q22.1 (B), R6.2
- new net: Q2.2 (B1), Q2.4 (E2)
- new net: C12.1, Q24.3 (E), Q26.1 (B), R1.2
- new net: Q21.2 (C), Q24.2 (C), Q26.2 (C), R1.1
- new net: Q17.1 (B), R5.1, R6.1
- new net: Q17.3 (E), Q18.2 (C)
- new net: Q2.1 (E1), Q2.3 (C2)
- new net: Q2.4 (E2), R5.1
- new net: Q2.2 (B1), Q2.4 (E2), Q2.5 (B2), Q2.6 (C1)
- new net: C12.2, Q2.3 (C2), Q24.1 (B), R1.1
- new net: Q2.2 (B1), Q2.4 (E2), R5.1
- new net: Q2.5 (B2), Q2.6 (C1), R6.1 (x2)
- new net: Q14.3 (E), Q18.1 (B), R5.2
- new net: Q14.2 (C), Q18.3 (E), Q2.3 (C2)
- new net: R5.1, RV2.3
- new net: Q1.2 (B1), Q1.4 (E2)
- new net: C14.2, Q1.5 (B2), R101.2
- new net: C1.1, R6.2, U1.2 (-)
- new net: Q1.3 (C2), Q13.2 (C), Q15.3 (E)
- new net: Q1.2 (B1), Q1.4 (E2), Q1.5 (B2), Q1.6 (C1)
- new net: C6.1, Q1.2 (B1), Q1.5 (B2), Q1.6 (C1), Q13.1 (B), Q5.2 (C)
- new net: Q22.2 (C), Q23.3 (E), Q25.3 (E), R1.2
- new net: Q22.3 (E), R1.2
- new net: C11.2, Q23.2 (C), Q25.1 (B), R1.1
- new net: Q3.2 (C), Q7.3 (E), R1.1
- new net: F2.1, J3.4 (Pin_4)
- new net: Q1.3 (C2), Q5.1 (B), R1.2
- new net: Q15.2 (C), Q16.3 (E)
- new net: C14.1, Q2.5 (B2), R101.2
- new net: C8.2, R1.1
- new net: Q2.1 (E1), R1.2
- new net: Q7.1 (B), R1.1, R1.2
- new net: Q7.2 (C), Q8.3 (E)
- new net: Q2.2 (B1), Q2.4 (E2), R8.1
- new net: R5.2, RV3.3
- new net: C7.2, Q14.1 (B), Q2.2 (B1), Q2.5 (B2), Q2.6 (C1), Q8.2 (C)
- new net: Q5.3 (E), Q6.2 (C)
- new net: Q4.2 (C), Q6.3 (E), R1.2
- new net: Q4.3 (E), R1.2
- new net: Q2.3 (C2), Q8.1 (B), R1.1
- new net: Q1.1 (E1), R1.1
- new net: C6.2, C8.1, R6.2
- new net: Q1.1 (E1), Q1.3 (C2)
- new net: Q1.4 (E2), R5.2
- new net: C2.2, R6.1, U1.3 (+)
- new net +18V: C14.1, C15.1, D1.1 (K), F1.2, Q1.1 (E1), Q2.3 (C2), Q2.6 (C1), Q25.2 (C), R1.2, R101.1, RV2.1, RV2.2
- new net -18V: C17.2, C18.2, D2.2 (A), F2.2, Q1.3 (C2), Q1.6 (C1), Q2.1 (E1), Q26.3 (E), R1.1, R101.1, RV3.1, RV3.2
- new net Amp_FB: R1.1, R1.1, R1.1, R1.2, R1.2
- new net Amp_Out: D1.2 (A), D2.1 (K), J2.2 (Pin_2), R1.1, R1.2, R1.2, R1.2, R6.1, R6.2, R6.2
- new net VCC: C14.1, C3.1, Q1.1 (E1), Q2.1 (E1), R1.2, R5.1, R5.1, U1.7 (V+)
- new net VEE: C14.2, C4.1, Q1.1 (E1), Q2.1 (E1), R1.1, R5.2, R8.2, U1.4 (V-)
- no-connect marks 0 -> 2
Other:
- removed sheet Amp L
- removed sheet Amp R
- removed sheet DC Protection
- note added: "Gain = 4.78"
- note added: "PGFB threshold = +14V"
